File: Achilles/input_board/adc.kicad_sch (KiCad schematic)
At the start: 14 parts, among them IC10 ADS8860IDGSR, U12 REF6050xDGK, U13 uA7805

Commit message: test version PCB
Parts:
- added TP16: REF_OUT, TestPoint:TestPoint_Keystone_5000-5004_Miniature, symbol Connector:TestPoint
- added TP17: CAL, TestPoint:TestPoint_Keystone_5000-5004_Miniature, symbol Connector:TestPoint
- added TP18: AINP, TestPoint:TestPoint_Keystone_5000-5004_Miniature, symbol Connector:TestPoint
- RN1: value MAX5490TA05000-T -> MAX5490GA01000-T
Connections:
- net CAL: now also TP17.1
- net REF_OUT: now also TP16.1
- net at R45.1, RN2.3 (R2): now also TP18.1
Other:
- note added: "100kR series Matched 1:1 ratio 0.035% ratio accuracy"
