File: Achilles/input_board/amplifiers.kicad_sch (KiCad schematic)
At the start: 28 parts, among them IC8 MUX36D08IPW, IC9 MUX508IPW, U10 INA849DGK, U11 INA849DGK, U4 INA849DGK, U5 INA849DGK, U6 INA849DGK, U7 INA849DGK, U8 INA849DGK, U9 INA849DGK

Commit message: test version PCB
Parts:
- added TP10: AMP2-, TestPoint:TestPoint_Keystone_5000-5004_Miniature, symbol Connector:TestPoint
- added TP11: AMP2+, TestPoint:TestPoint_Keystone_5000-5004_Miniature, symbol Connector:TestPoint
- added TP12: A2_OUT, TestPoint:TestPoint_Keystone_5000-5004_Miniature, symbol Connector:TestPoint
- added TP13: AMP3-, TestPoint:TestPoint_Keystone_5000-5004_Miniature, symbol Connector:TestPoint
- added TP14: AMP3+, TestPoint:TestPoint_Keystone_5000-5004_Miniature, symbol Connector:TestPoint
- added TP15: A3_OUT, TestPoint:TestPoint_Keystone_5000-5004_Miniature, symbol Connector:TestPoint
- added TP24: AMPS0, TestPoint:TestPoint_Keystone_5000-5004_Miniature, symbol Connector:TestPoint
- added TP25: AMPS1, TestPoint:TestPoint_Keystone_5000-5004_Miniature, symbol Connector:TestPoint
- added TP26: AMPS2, TestPoint:TestPoint_Keystone_5000-5004_Miniature, symbol Connector:TestPoint
- added TP27, TP28: AMPIN-, TestPoint:TestPoint_Keystone_5000-5004_Miniature, symbol Connector:TestPoint
- added TP7: A1_OUT, TestPoint:TestPoint_Keystone_5000-5004_Miniature, symbol Connector:TestPoint
- added TP8: AMP1-, TestPoint:TestPoint_Keystone_5000-5004_Miniature, symbol Connector:TestPoint
- added TP9: AMP1+, TestPoint:TestPoint_Keystone_5000-5004_Miniature, symbol Connector:TestPoint
Connections:
- net A1_OUT: now also TP7.1
- net A2_OUT: now also TP12.1
- net A3_OUT: now also TP15.1
- net AMP1+: now also TP9.1
- net AMP1-: now also TP8.1
- net AMP2+: now also TP11.1
- net AMP2-: now also TP10.1
- net AMP3+: now also TP14.1
- net AMP3-: now also TP13.1
- net AMP_IN+: now also TP28.1
- net AMP_IN-: now also TP27.1
- net AMP_SEL_0: now also TP24.1
- net AMP_SEL_1: now also TP25.1
- net AMP_SEL_2: now also TP26.1
