File: Achilles/input_board/frontend.kicad_sch (KiCad schematic)
At the start: 30 parts, among them IC2 TMUX7349FPWR, IC3 TMUX7349FPWR, IC4 TMUX7349FPWR, IC5 TMUX7349FPWR, IC6 MUX509IPW, IC7 MUX509IPW, J11 Screw_Terminal_01x02, J3 Screw_Terminal_01x08, J4 Screw_Terminal_01x08, J5 Screw_Terminal_01x08, J6 Screw_Terminal_01x08, J7 Screw_Terminal_01x02

Commit message: test version PCB
Parts:
- added TP19: IN_A0, TestPoint:TestPoint_Keystone_5000-5004_Miniature, symbol Connector:TestPoint
- added TP20: IN_A1, TestPoint:TestPoint_Keystone_5000-5004_Miniature, symbol Connector:TestPoint
- added TP21: SF_1..4, TestPoint:TestPoint_Keystone_5000-5004_Miniature, symbol Connector:TestPoint
- added TP22: FF_1..4, TestPoint:TestPoint_Keystone_5000-5004_Miniature, symbol Connector:TestPoint
- added TP23: EN, TestPoint:TestPoint_Keystone_5000-5004_Miniature, symbol Connector:TestPoint
- added TP29: SEL_IN_2, TestPoint:TestPoint_Keystone_5000-5004_Miniature, symbol Connector:TestPoint
- added TP30: SEL_IN_3, TestPoint:TestPoint_Keystone_5000-5004_Miniature, symbol Connector:TestPoint
Connections:
- net FAULT_1..4: now also TP22.1
- net INPUT_EN: now also TP23.1
- net SEL_IN_0: now also TP19.1
- net SEL_IN_1: now also TP20.1
- net SEL_IN_2: now also TP29.1
- net SEL_IN_3: now also TP30.1
- net SF_1..4: now also TP21.1
Other:
- moved on the sheet: C20, C21, C24, IC4, IC7, R27, R28
