File: Automedon/automedon/daq.kicad_sch (KiCad schematic)
At the start: 16 parts, among them J17 09-4224-00-04, J18 09-4224-00-04, J19 09-4224-00-04, J20 09-4224-00-04, J21 09-4224-00-04, J22 09-4224-00-04, J23 09-4224-00-04, J24 09-4224-00-04, J25 09-4224-00-04, J26 09-4224-00-04, J27 09-4224-00-04, J28 09-4224-00-04

Commit message: Revert other files to main
Changed lines of the file:
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@@
 (kicad_sch
-	(version 20250114)
+	(version 20231120)
 	(generator "eeschema")
-	(generator_version "9.0")
+	(generator_version "8.0")
 	(paper "A3")
-	(rectangle
-		(start 44.45 215.9)
-		(end 207.01 266.7)
-		(stroke
-			(width 0)
-			(type default)
-		)
-		(fill
-			(type none)
-		)
-	)
-	(rectangle
-		(start 107.315 46.99)
-		(end 260.985 197.485)
-		(stroke
-			(width 0)
-			(type default)
-		)
-		(fill
-			(type none)
-		)
-	)
-	(rectangle
-		(start 233.045 221.615)
-		(end 280.035 267.97)
-		(stroke
-			(width 0)
-			(type default)
-		)
-		(fill
-			(type none)
-		)
-	)
-	(text "RasPi"
-		(exclude_from_sim no)
-		(at 252.476 234.696 0)
-		(effects
-			(font
-				(size 1.27 1.27)
-			)
-		)
-	)
-	(text "Low-Noise Supplies"
-		(exclude_from_sim no)
-		(at 122.428 242.316 0)
-		(effects
-			(font
-				(size 1.27 1.27)
-			)
-		)
-	)
-	(text "NI Box"
-		(exclude_from_sim no)
-		(at 183.642 133.35 0)
-		(effects
-			(font
-				(size 1.27 1.27)
-			)
-		)
-	)
 	(no_connect
 		(at 290.83 187.96)
@@
 		)
 	)
+	(rectangle
+		(start 44.45 215.9)
+		(end 207.01 266.7)
+		(stroke
+			(width 0)
+			(type default)
+		)
+		(fill
+			(type none)
+		)
+	)
+	(rectangle
+		(start 107.315 46.99)
+		(end 260.985 197.485)
+		(stroke
+			(width 0)
+			(type default)
+		)
+		(fill
+			(type none)
+		)
+	)
+	(rectangle
+		(start 233.045 221.615)
+		(end 280.035 267.97)
+		(stroke
+			(width 0)
+			(type default)
+		)
+		(fill
+			(type none)
+		)
+	)
+	(text "RasPi"
+		(exclude_from_sim no)
+		(at 252.476 234.696 0)
+		(effects
+			(font
+				(size 1.27 1.27)
+			)
+		)
+	)
+	(text "Low-Noise Supplies"
+		(exclude_from_sim no)
+		(at 122.428 242.316 0)
+		(effects
+			(font
+				(size 1.27 1.27)
+			)
+		)
+	)
+	(text "NI Box"
+		(exclude_from_sim no)
+		(at 183.642 133.35 0)
+		(effects
+			(font
+				(size 1.27 1.27)
+			)
+		)
+	)

Commit message: Update KiCad schematics and add power converter library
Changed lines of the file:
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@@
 (kicad_sch
-	(version 20231120)
+	(version 20250114)
 	(generator "eeschema")
-	(generator_version "8.0")
+	(generator_version "9.0")
 	(paper "A3")
+	(rectangle
+		(start 44.45 215.9)
+		(end 207.01 266.7)
+		(stroke
+			(width 0)
+			(type default)
+		)
+		(fill
+			(type none)
+		)
+	)
+	(rectangle
+		(start 107.315 46.99)
+		(end 260.985 197.485)
+		(stroke
+			(width 0)
+			(type default)
+		)
+		(fill
+			(type none)
+		)
+	)
+	(rectangle
+		(start 233.045 221.615)
+		(end 280.035 267.97)
+		(stroke
+			(width 0)
+			(type default)
+		)
+		(fill
+			(type none)
+		)
+	)
+	(text "RasPi"
+		(exclude_from_sim no)
+		(at 252.476 234.696 0)
+		(effects
+			(font
+				(size 1.27 1.27)
+			)
+		)
+	)
+	(text "Low-Noise Supplies"
+		(exclude_from_sim no)
+		(at 122.428 242.316 0)
+		(effects
+			(font
+				(size 1.27 1.27)
+			)
+		)
+	)
+	(text "NI Box"
+		(exclude_from_sim no)
+		(at 183.642 133.35 0)
+		(effects
+			(font
+				(size 1.27 1.27)
+			)
+		)
+	)
 	(no_connect
 		(at 290.83 187.96)
@@
 		)
 	)
-	(rectangle
-		(start 44.45 215.9)
-		(end 207.01 266.7)
-		(stroke
-			(width 0)
-			(type default)
-		)
-		(fill
-			(type none)
-		)
-	)
-	(rectangle
-		(start 107.315 46.99)
-		(end 260.985 197.485)
-		(stroke
-			(width 0)
-			(type default)
-		)
-		(fill
-			(type none)
-		)
-	)
-	(rectangle
-		(start 233.045 221.615)
-		(end 280.035 267.97)
-		(stroke
-			(width 0)
-			(type default)
-		)
-		(fill
-			(type none)
-		)
-	)
-	(text "RasPi"
-		(exclude_from_sim no)
-		(at 252.476 234.696 0)
-		(effects
-			(font
-				(size 1.27 1.27)
-			)
-		)
-	)
-	(text "Low-Noise Supplies"
-		(exclude_from_sim no)
-		(at 122.428 242.316 0)
-		(effects
-			(font
-				(size 1.27 1.27)
-			)
-		)
-	)
-	(text "NI Box"
-		(exclude_from_sim no)
-		(at 183.642 133.35 0)
-		(effects
-			(font
-				(size 1.27 1.27)
-			)
-		)
-	)
