File: Automedon/automedon/daq.kicad_sch (KiCad schematic)
At the start: 16 parts, among them J17 09-4224-00-04, J18 09-4224-00-04, J19 09-4224-00-04, J20 09-4224-00-04, J21 09-4224-00-04, J22 09-4224-00-04, J23 09-4224-00-04, J24 09-4224-00-04, J25 09-4224-00-04, J26 09-4224-00-04, J27 09-4224-00-04, J28 09-4224-00-04

Commit message: Update bunch of other stuff - dont touch power
Parts:
- added U19: USB POWER, symbol automedon:USB_PWR
- added U20, U21, U22: DAQ PWR, symbol automedon:DAQ_PWR
Connections:
- net DAQ_12: now also U21. (GND)
- net DAQ_24: now also U20. (GND)
- net DAQ_5: now also U22. (GND)
- net GND: now also U19. (USB_C), U20. (GND), U21. (GND), U22. (GND)
- new net +12V: U19. (USB_C)
- new net +24V: U20. (GND), U21. (GND), U22. (GND)
- new net 12_MON: U21. (GND)
- new net 24_MON: U20. (GND)
- new net 5_MON: U22. (GND)
- no-connect marks 4 -> 14
Other:
- note added: "12V @ 3A"
- note added: "LINK"
- note added: "LabJack T7"
- note removed: "Low-Noise Supplies"
- note removed: "NI Box"
