File: Automedon/automedon/ethernet.kicad_sch (KiCad schematic)
At the start: 2 parts

Commit message: Revert other files to main
Connections:
- new net: U10. (GND), U11. (VIN-)
Changed lines of the file:
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@@
 (kicad_sch
-	(version 20250114)
+	(version 20231120)
 	(generator "eeschema")
-	(generator_version "9.0")
+	(generator_version "8.0")
 	(paper "A4")
-	(text "TP-DCDC-1224G"
-		(exclude_from_sim no)
-		(at 157.226 80.01 0)
-		(effects
-			(font
-				(size 1.27 1.27)
-			)
-		)
-	)
-	(text "2W @ 12V"
-		(exclude_from_sim no)
-		(at 103.632 99.06 0)
-		(effects
-			(font
-				(size 1.27 1.27)
-			)
-		)
-	)
-	(text "Ubiquiti LiteBeam takes max 0.3A @ 24V"
-		(exclude_from_sim no)
-		(at 164.338 94.996 0)
-		(effects
-			(font
-				(size 1.27 1.27)
-			)
-		)
-	)
-	(text "SE-SW5U-WT"
-		(exclude_from_sim no)
-		(at 103.886 80.01 0)
-		(effects
-			(font
-				(size 1.27 1.27)
-			)
-		)
-	)
 	(wire
 		(pts
@@
 		)
 	)
+	(text "TP-DCDC-1224G"
+		(exclude_from_sim no)
+		(at 157.226 80.01 0)
+		(effects
+			(font
+				(size 1.27 1.27)
+			)
+		)
+	)
+	(text "2W @ 12V"
+		(exclude_from_sim no)
+		(at 103.632 99.06 0)
+		(effects
+			(font
+				(size 1.27 1.27)
+			)
+		)
+	)
+	(text "Ubiquiti LiteBeam takes max 0.3A @ 24V"
+		(exclude_from_sim no)
+		(at 164.338 94.996 0)
+		(effects
+			(font
+				(size 1.27 1.27)
+			)
+		)
+	)
+	(text "SE-SW5U-WT"
+		(exclude_from_sim no)
+		(at 103.886 80.01 0)
+		(effects
+			(font
+				(size 1.27 1.27)
+			)
+		)
+	)

Commit message: Update KiCad schematics and add power converter library
Connections:
- new net: U10. (ETH_OUT), U11. (ETH_5)
Changed lines of the file:
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@@
 (kicad_sch
-	(version 20231120)
+	(version 20250114)
 	(generator "eeschema")
-	(generator_version "8.0")
+	(generator_version "9.0")
 	(paper "A4")
+	(text "TP-DCDC-1224G"
+		(exclude_from_sim no)
+		(at 157.226 80.01 0)
+		(effects
+			(font
+				(size 1.27 1.27)
+			)
+		)
+	)
+	(text "2W @ 12V"
+		(exclude_from_sim no)
+		(at 103.632 99.06 0)
+		(effects
+			(font
+				(size 1.27 1.27)
+			)
+		)
+	)
+	(text "Ubiquiti LiteBeam takes max 0.3A @ 24V"
+		(exclude_from_sim no)
+		(at 164.338 94.996 0)
+		(effects
+			(font
+				(size 1.27 1.27)
+			)
+		)
+	)
+	(text "SE-SW5U-WT"
+		(exclude_from_sim no)
+		(at 103.886 80.01 0)
+		(effects
+			(font
+				(size 1.27 1.27)
+			)
+		)
+	)
 	(wire
 		(pts
@@
 		)
 	)
-	(text "TP-DCDC-1224G"
-		(exclude_from_sim no)
-		(at 157.226 80.01 0)
-		(effects
-			(font
-				(size 1.27 1.27)
-			)
-		)
-	)
-	(text "2W @ 12V"
-		(exclude_from_sim no)
-		(at 103.632 99.06 0)
-		(effects
-			(font
-				(size 1.27 1.27)
-			)
-		)
-	)
-	(text "Ubiquiti LiteBeam takes max 0.3A @ 24V"
-		(exclude_from_sim no)
-		(at 164.338 94.996 0)
-		(effects
-			(font
-				(size 1.27 1.27)
-			)
-		)
-	)
-	(text "SE-SW5U-WT"
-		(exclude_from_sim no)
-		(at 103.886 80.01 0)
-		(effects
-			(font
-				(size 1.27 1.27)
-			)
-		)
-	)
