File: Automedon/automedon/ethernet.kicad_sch (KiCad schematic)
At the start: 2 parts

Commit message: Update eth subsheet
Parts:
- removed U10: ~, symbol automedon:POE_INJ
- removed U11: ~, symbol automedon:ETH_SW
- added U10: DS108G-M2, symbol automedon:ETH_SW
- added U11: ER605v2, symbol automedon:ETH_ROUTER
- added U18: OC200, symbol automedon:ETH_HW_CTL
- added U19: USB HUB, symbol automedon:USB_PWR
Connections:
- net +12V: now also U10. (ETH_8), U11. (LAN2), U19. (USB_4)
- net ANTENNA_ETH: now also U10. (ETH_8)
- net ETH_DAQ: now also U10. (ETH_8)
- net ETH_DEBUG: now also U10. (ETH_8)
- net ETH_PI: now also U10. (ETH_8)
- net ETH_RLCS: now also U10. (ETH_8)
- net GND: now also U10. (ETH_8), U11. (LAN2), U19. (USB_4)
- new net ETH_WAP: U10. (ETH_8)
- new net OC_200_PWR: U18. (ETH_2), U19. (USB_4)
- new net PI_USB: U19. (USB_4)
- new net T7_USB: U19. (USB_4)
- no-connect marks 0 -> 10
Other:
- note added: "12V @ 1A (barrel jack)"
- note added: "12V @ 3A"
- note added: "DS108G (NON P)"
- note added: "PART LINK"
- note removed: "2W @ 12V"
- note removed: "SE-SW5U-WT"
- note removed: "TP-DCDC-1224G"
- note removed: "Ubiquiti LiteBeam takes max 0.3A @ 24V"
