File: Automedon/automedon/automedon.kicad_sch (KiCad schematic)
At the start: 10 parts, among them J1 701W-X2/03, J13 ZP-PNA-06-101, J16 Antenna, J2 MS3100E24-22P, J3 PWM-02RMFS-TS7001, J4 PWM-02RMFS-TS7001, J45 PWM-02RMFS-TS7001, SW1 RB242D1021-117/ACC-F02-1, SW3 KEYSWITCH_SPST

Commit message: Update bunch of other stuff - dont touch power
Parts:
- removed J13: ZP-PNA-06-101, symbol Connector:Conn_01x01_Socket
- removed J16: Antenna, symbol Connector:Conn_01x01_Socket
- added J5: Antenna, symbol Connector:Conn_01x08_Socket
- added J6: WAP, symbol Connector:Conn_01x08_Socket
- SW1: value RB242D1021-117/ACC-F02-1 -> RRS20F1ABLKREDBLK31P
Connections:
- new net +24V: J5.4 (Pin_4), J5.5 (Pin_5), J6.4 (Pin_4), J6.5 (Pin_5)
- new net GND: J5.7 (Pin_7), J5.8 (Pin_8), J6.7 (Pin_7), J6.8 (Pin_8)
- new net ethernet/ETH_ANTENNA: J5.1 (Pin_1), J5.2 (Pin_2), J5.3 (Pin_3), J5.6 (Pin_6)
- new net ethernet/ETH_WAP: J6.1 (Pin_1), J6.2 (Pin_2), J6.3 (Pin_3), J6.6 (Pin_6)
Other:
- sheet daq ports: added ETH_DAQ, ETH_PI, OC_200_PWR; removed none
- sheet ethernet ports: added ETH_ANTENNA, ETH_PI, ETH_WAP, OC_200_PWR; removed ANTENNA_ETH, ETH_DEBUG
- note added: "TPLINK WAP is Passive PoE 2-pair (4, 5+; 7, 8 return)"
- note added: "Ubiquiti Antenna is Passive PoE 2-pair (4, 5+; 7, 8 return)"
- note removed: "*Rated to 15A but IP67"
- note removed: "Antenna is Passive PoE 2-pair (4, 5+; 7, 8 return)"
- note removed: "Debug Port"
- note removed: "M12 X-coded"
