File: Automedon/automedon/tank_heating.kicad_sch (KiCad schematic)
At the start: 3 parts

Commit message: Update KiCad schematics and add power converter library
Connections:
- net at U3. (SDA/CANL): no longer U1. (SDA/CANL)
- new net: U1. (SDA/CANL), U3. (SDA/CANL) (x5)
- new net: U1.1 (ACT_GND), U3.1 (ACT_GND) (x2)
- new net: U1.1 (ACT_GND), U2. (GND) (x2)
- now unconnected: U3. (SDA/CANL), U3. (SDA/CANL), U3. (SDA/CANL), U3. (SDA/CANL)

Commit message: Revert other files to main
Connections:
- net at U3. (SDA/CANL): no longer U1. (SDA/CANL)
- new net: U1. (SDA/CANL), U3. (SDA/CANL) (x5)
- new net: U1.1 (P1), U3.1 (P1) (x2)
- new net: U1.1 (P1), U2. (VOUT) (x2)
- now unconnected: U3. (SDA/CANL), U3. (SDA/CANL), U3. (SDA/CANL), U3. (SDA/CANL)
