File: Automedon/automedon/tank_heating.kicad_sch (KiCad schematic)
At the start: 3 parts

Commit message: Update a bunch of shit
Parts:
- added J59, J60: 32xxx, symbol automedon:CONN_TERM_3
- added U35: ~, symbol automedon:RPP
Connections:
- net BATT_24+: now also J59.1; no longer U2. (GND)
- net BATT_24-: now also J60.1; no longer U2. (GND)
- net at U3. (SDA/CANL): no longer U1. (SDA/CANL)
- net at U2. (GND): now also J60.1; no longer U1.1 (ACT_GND)
- new net: U1. (SDA/CANL), U3. (SDA/CANL) (x5)
- new net: U1.1 (ACT_GND), U2. (GND) (x2)
- new net: J59.1, U35. (GND)
- new net: J59.1, U2. (GND)
- new net: U3.1 (ACT_GND), U35. (GND) (x2)
- new net: J60.1, U35. (GND)
- now unconnected: U3. (SDA/CANL), U3. (SDA/CANL), U3. (SDA/CANL), U3. (SDA/CANL)
- no-connect marks 13 -> 15
Other:
- note removed: "add 3rd?"
