File: Automedon/automedon/valve_relays.kicad_sch (KiCad schematic)
At the start: 17 parts, among them J10 MS3102E14S-6S, J11 MS3102E14S-6S, J12 MS3102E14S-6S, J14 Conn_01x02_Pin, J15 Conn_01x02_Pin, J7 MS3102E14S-6S, J8 MS3102E14S-6S, J9 MS3102E14S-6S, SW2 SW_DPST_x2

Commit message: Update KiCad schematics and add power converter library
Connections:
- net at U5. (SDA/CANL): now also U6. (SDA/CANL); no longer U4. (SDA/CANL)
- net at U5.1 (ACT_GND): now also J8.1 (Pin_1); no longer U4.1 (P1)
- net at U6. (SDA/CANL): now also U7. (SDA/CANL); no longer U5. (SDA/CANL)
- net at U6.1 (ACT_GND): now also U7.1 (ACT_GND); no longer U5.1 (P1)
- net at U9. (SDA/CANL): now also U8. (SDA/CANL)
- net at U8. (SDA/CANL): now also U7. (SDA/CANL); no longer U9. (SDA/CANL)
- net at U9.1 (ACT_GND): now also J12.1 (Pin_1)
- net at U8.1 (ACT_GND): now also U7.1 (ACT_GND); no longer U9.1 (P1)
- new net: U4. (SDA/CANL), U5. (SDA/CANL) (x5)
- new net: U12. (SDA/CANL), U4. (SDA/CANL) (x2)
- new net: U4.1 (ACT_GND), U5.1 (ACT_GND) (x2)
- new net: U5. (SDA/CANL), U6. (SDA/CANL) (x4)
- new net: U5.1 (ACT_GND), U6.1 (ACT_GND) (x2)
- new net: U8. (SDA/CANL), U9. (SDA/CANL) (x4)
- new net: U8.1 (ACT_GND), U9.1 (ACT_GND) (x2)
- new net: U6. (SDA/CANL), U7. (SDA/CANL) (x4)
- new net: U7. (SDA/CANL), U8. (SDA/CANL) (x4)
- new net: U6.1 (ACT_GND), U7.1 (ACT_GND)
- new net: U7.1 (ACT_GND), U8.1 (ACT_GND)

Commit message: Revert other files to main
Connections:
- net at U5. (SDA/CANL): now also U6. (SDA/CANL); no longer U4. (SDA/CANL)
- net at U5.1 (P1): now also J8.1 (Pin_1); no longer U4.1 (ACT_GND)
- net at U6. (SDA/CANL): now also U7. (SDA/CANL); no longer U5. (SDA/CANL)
- net at U6.1 (P1): now also U7.1 (P1); no longer U5.1 (ACT_GND)
- net at U9. (SDA/CANL): now also U8. (SDA/CANL)
- net at U8. (SDA/CANL): now also U7. (SDA/CANL); no longer U9. (SDA/CANL)
- net at U9.1 (P1): now also J12.1 (Pin_1)
- net at U8.1 (P1): now also U7.1 (P1); no longer U9.1 (ACT_GND)
- new net: U4. (SDA/CANL), U5. (SDA/CANL) (x5)
- new net: U12. (UART_TX), U4. (SDA/CANL) (x2)
- new net: U4.1 (P1), U5.1 (P1) (x2)
- new net: U5. (SDA/CANL), U6. (SDA/CANL) (x4)
- new net: U5.1 (P1), U6.1 (P1) (x2)
- new net: U8. (SDA/CANL), U9. (SDA/CANL) (x4)
- new net: U8.1 (P1), U9.1 (P1) (x2)
- new net: U6. (SDA/CANL), U7. (SDA/CANL) (x4)
- new net: U7. (SDA/CANL), U8. (SDA/CANL) (x4)
- new net: U6.1 (P1), U7.1 (P1)
- new net: U7.1 (P1), U8.1 (P1)
